File: adc.sch (KiCad schematic (older format))
At the start: 55 parts, among them J1 Conn_01x08_Male, J2 Conn_01x06_Male, J3 Conn_01x08_Male, J4 Conn_01x10_Male, J5 Conn_02x08_Top_Bottom, J6 Conn_02x08_Top_Bottom, J7 Conn_02x08_Top_Bottom, U1 ADC128D818, U2 ADC128D818, U3 ADC128D818

Commit message: rev 0
Parts:
- removed C5, C7: 1U ELEC, Capacitors_SMD:CP_Elec_5x5.8, symbol Device:CP
- removed J5, J6, J7: Conn_02x08_Top_Bottom, Socket_Strips:Socket_Strip_Straight_2x08_Pitch2.54mm, symbol Connector_Generic:Conn_02x08_Top_Bottom
- added J5, J6, J7: Conn_02x08_Odd_Even, Socket_Strips:Socket_Strip_Straight_2x08_Pitch2.54mm, symbol Connector_Generic:Conn_02x08_Odd_Even
- A1: footprint Module:Arduino_UNO_R3 -> Footprints:Arduino_UNO_R3
- U1, U2, U3: footprint Package_SO:TSSOP-16_4.4x5mm_P0.65mm -> Footprints:TSSOP-16_4.4x5mm_P0.65mm
Connections:
- net GND: now also J5.10 (Pin_10), J5.12 (Pin_12), J5.14 (Pin_14), J5.16 (Pin_16), J5.2 (Pin_2), J5.4 (Pin_4), J5.6 (Pin_6), J5.8 (Pin_8), J6.10 (Pin_10), J6.12 (Pin_12), J6.14 (Pin_14), J6.16 (Pin_16), J6.2 (Pin_2), J6.4 (Pin_4), J6.6 (Pin_6), J6.8 (Pin_8), J7.10 (Pin_10), J7.12 (Pin_12), J7.14 (Pin_14), J7.16 (Pin_16), J7.2 (Pin_2), J7.4 (Pin_4), J7.6 (Pin_6), J7.8 (Pin_8)
- net at R11.2, U1.10 (IN6): now also J5.13 (Pin_13)
- net at R10.2, U1.11 (IN5): now also J5.11 (Pin_11)
- net at R9.2, U1.12 (IN4): now also J5.9 (Pin_9)
- net at R8.2, U1.13 (IN3): now also J5.7 (Pin_7)
- net at R7.2, U1.14 (IN2): now also J5.5 (Pin_5)
- net at R6.2, U1.15 (IN1): now also J5.3 (Pin_3)
- net at R4.2, U1.16 (IN0): now also J5.1 (Pin_1)
- net at R12.2, U1.9 (IN7): now also J5.15 (Pin_15)
- net at R31.2, U3.10 (IN6): now also J7.13 (Pin_13)
- net at R30.2, U3.11 (IN5): now also J7.11 (Pin_11)
- net at R29.2, U3.12 (IN4): now also J7.9 (Pin_9)
- net at R28.2, U3.13 (IN3): now also J7.7 (Pin_7)
- net at R26.2, U3.14 (IN2): now also J7.5 (Pin_5)
- net at R24.2, U3.15 (IN1): now also J7.3 (Pin_3)
- net at R21.2, U3.16 (IN0): now also J7.1 (Pin_1)
- net at R32.2, U3.9 (IN7): now also J7.15 (Pin_15)
- net at R25.2, U2.10 (IN6): now also J6.13 (Pin_13)
- net at R22.2, U2.11 (IN5): now also J6.11 (Pin_11)
- net at R19.2, U2.12 (IN4): now also J6.9 (Pin_9)
- net at R18.2, U2.13 (IN3): now also J6.7 (Pin_7)
- net at R17.2, U2.14 (IN2): now also J6.5 (Pin_5)
- net at R16.2, U2.15 (IN1): now also J6.3 (Pin_3)
- net at R14.2, U2.16 (IN0): now also J6.1 (Pin_1)
- net at R27.2, U2.9 (IN7): now also J6.15 (Pin_15)
Changed lines of the file:
@@
 F 0 "U1" H 1750 3378 50  0000 C CNN
 F 1 "ADC128D818" H 1750 3287 50  0000 C CNN
-F 2 "Package_SO:TSSOP-16_4.4x5mm_P0.65mm" H 1750 2400 50  0001 C CIN
+F 2 "Footprints:TSSOP-16_4.4x5mm_P0.65mm" H 1750 2400 50  0001 C CIN
 F 3 "http://www.ti.com/lit/ds/symlink/adc128d818.pdf" H 1750 2400 50  0001 C CNN
 	1    1750 2400
 	-1   0    0    -1
-$EndComp
-$Comp
-L Connector_Generic:Conn_02x08_Top_Bottom J5
-U 1 1 5BF31AB7
-P 4450 2100
-F 0 "J5" H 4500 2617 50  0000 C CNN
-F 1 "Conn_02x08_Top_Bottom" H 4500 2526 50  0000 C CNN
-F 2 "Socket_Strips:Socket_Strip_Straight_2x08_Pitch2.54mm" H 4450 2100 50  0001 C CNN
-F 3 "~" H 4450 2100 50  0001 C CNN
-	1    4450 2100
-	1    0    0    -1
 $EndComp
 Wire Wire Line
@@
 F 0 "A1" H 2050 7728 50  0000 C CNN
 F 1 "Arduino_UNO_R3" H 2050 7637 50  0000 C CNN
-F 2 "Module:Arduino_UNO_R3" H 2200 5500 50  0001 L CNN
+F 2 "Footprints:Arduino_UNO_R3" H 2200 5500 50  0001 L CNN
 F 3 "https://www.arduino.cc/en/Main/arduinoBoardUno" H 1850 7600 50  0001 C CNN
 	1    2050 6550
@@
 F 0 "U3" H 6650 3428 50  0000 C CNN
 F 1 "ADC128D818" H 6650 3337 50  0000 C CNN
-F 2 "Package_SO:TSSOP-16_4.4x5mm_P0.65mm" H 6650 2450 50  0001 C CIN
+F 2 "Footprints:TSSOP-16_4.4x5mm_P0.65mm" H 6650 2450 50  0001 C CIN
 F 3 "http://www.ti.com/lit/ds/symlink/adc128d818.pdf" H 6650 2450 50  0001 C CNN
 	1    6650 2450
 	-1   0    0    -1
-$EndComp
-$Comp
-L Connector_Generic:Conn_02x08_Top_Bottom J7
-U 1 1 5BF7FD84
-P 9350 2150
-F 0 "J7" H 9400 2667 50  0000 C CNN
-F 1 "Conn_02x08_Top_Bottom" H 9400 2576 50  0000 C CNN
-F 2 "Socket_Strips:Socket_Strip_Straight_2x08_Pitch2.54mm" H 9350 2150 50  0001 C CNN
-F 3 "~" H 9350 2150 50  0001 C CNN
-	1    9350 2150
-	1    0    0    -1
 $EndComp
 Wire Wire Line
@@
 	6650 800  6650 1650
 $Comp
-L Device:CP C7
-U 1 1 5BF7FE6A
-P 6300 950
-F 0 "C7" H 6418 996 50  0000 L CNN
-F 1 "1U ELEC" H 6418 905 50  0000 L CNN
-F 2 "Capacitors_SMD:CP_Elec_5x5.8" H 6338 800 50  0001 C CNN
-F 3 "~" H 6300 950 50  0001 C CNN
-	1    6300 950
-	1    0    0    -1
-$EndComp
-Wire Wire Line
-	6300 800  6650 800
-$Comp
-L power:GND #PWR019
-U 1 1 5BF7FE72
-P 6300 1150
-F 0 "#PWR019" H 6300 900 50  0001 C CNN
-F 1 "GND" H 6305 977 50  0000 C CNN
-F 2 "" H 6300 1150 50  0001 C CNN
-F 3 "" H 6300 1150 50  0001 C CNN
-	1    6300 1150
-	1    0    0    -1
-$EndComp
-$Comp
 L power:GND #PWR023
 U 1 1 5BF7FE78
@@
 Wire Wire Line
 	6900 1100 6900 1150
-Wire Wire Line
-	6300 1100 6300 1150
 Text Label 6650 1250 1    50   ~ 0
 VIN
@@
 F 0 "U2" H 5650 6378 50  0000 C CNN
 F 1 "ADC128D818" H 5650 6287 50  0000 C CNN
-F 2 "Package_SO:TSSOP-16_4.4x5mm_P0.65mm" H 5650 5400 50  0001 C CIN
+F 2 "Footprints:TSSOP-16_4.4x5mm_P0.65mm" H 5650 5400 50  0001 C CIN
 F 3 "http://www.ti.com/lit/ds/symlink/adc128d818.pdf" H 5650 5400 50  0001 C CNN
 	1    5650 5400
 	-1   0    0    -1
-$EndComp
-$Comp
-L Connector_Generic:Conn_02x08_Top_Bottom J6
-U 1 1 5BFE99A1
-P 8350 5100
-F 0 "J6" H 8400 5617 50  0000 C CNN
-F 1 "Conn_02x08_Top_Bottom" H 8400 5526 50  0000 C CNN
-F 2 "Socket_Strips:Socket_Strip_Straight_2x08_Pitch2.54mm" H 8350 5100 50  0001 C CNN
-F 3 "~" H 8350 5100 50  0001 C CNN
-	1    8350 5100
-	1    0    0    -1
 $EndComp
 Wire Wire Line
@@
 	5650 3750 5650 4600
 $Comp
-L Device:CP C5
-U 1 1 5BFE9A79
-P 5300 3900
-F 0 "C5" H 5418 3946 50  0000 L CNN
-F 1 "1U ELEC" H 5418 3855 50  0000 L CNN
-F 2 "Capacitors_SMD:CP_Elec_5x5.8" H 5338 3750 50  0001 C CNN
-F 3 "~" H 5300 3900 50  0001 C CNN
-	1    5300 3900
-	1    0    0    -1
-$EndComp
-Wire Wire Line
-	5300 3750 5650 3750
-$Comp
-L power:GND #PWR014
-U 1 1 5BFE9A81
-P 5300 4100
-F 0 "#PWR014" H 5300 3850 50  0001 C CNN
-F 1 "GND" H 5305 3927 50  0000 C CNN
-F 2 "" H 5300 4100 50  0001 C CNN
-F 3 "" H 5300 4100 50  0001 C CNN
-	1    5300 4100
-	1    0    0    -1
-$EndComp
-$Comp
 L power:GND #PWR017
 U 1 1 5BFE9A87
@@
 Wire Wire Line
 	5900 4050 5900 4100
-Wire Wire Line
-	5300 4050 5300 4100
 Text Label 5650 4200 1    50   ~ 0
 VIN
@@
 Wire Wire Line
 	1250 6250 1250 6200
+$Comp
+L Connector_Generic:Conn_02x08_Odd_Even J5
+U 1 1 5C07D8AC
+P 4450 2100
+F 0 "J5" H 4500 2617 50  0000 C CNN
+F 1 "Conn_02x08_Odd_Even" H 4500 2526 50  0000 C CNN
+F 2 "Socket_Strips:Socket_Strip_Straight_2x08_Pitch2.54mm" H 4450 2100 50  0001 C CNN
+F 3 "~" H 4450 2100 50  0001 C CNN
+	1    4450 2100
+	1    0    0    -1
+$EndComp
+$Comp
+L Connector_Generic:Conn_02x08_Odd_Even J7
+U 1 1 5C07DA7D
+P 9350 2150
+F 0 "J7" H 9400 2667 50  0000 C CNN
+F 1 "Conn_02x08_Odd_Even" H 9400 2576 50  0000 C CNN
+F 2 "Socket_Strips:Socket_Strip_Straight_2x08_Pitch2.54mm" H 9350 2150 50  0001 C CNN
+F 3 "~" H 9350 2150 50  0001 C CNN
+	1    9350 2150
+	1    0    0    -1
+$EndComp
+$Comp
+L Connector_Generic:Conn_02x08_Odd_Even J6
+U 1 1 5C07E2C2
+P 8350 5100
+F 0 "J6" H 8400 5617 50  0000 C CNN
+F 1 "Conn_02x08_Odd_Even" H 8400 5526 50  0000 C CNN
+F 2 "Socket_Strips:Socket_Strip_Straight_2x08_Pitch2.54mm" H 8350 5100 50  0001 C CNN
+F 3 "~" H 8350 5100 50  0001 C CNN
+	1    8350 5100
+	1    0    0    -1
+$EndComp
 $EndSCHEMATC

Commit message: misc
Parts:
- removed A1: Arduino_UNO_R3, Footprints:Arduino_UNO_R3, symbol MCU_Module:Arduino_UNO_R3
Connections:
- net VCC: no longer J1.8 (Pin_8)
- no-connect marks 4 -> 5
Other:
- moved on the sheet: J3, J4
Changed lines of the file:
@@
 Connection ~ 4800 1900
-$Comp
-L MCU_Module:Arduino_UNO_R3 A1
-U 1 1 5BF3D2A7
-P 2050 6550
-F 0 "A1" H 2050 7728 50  0000 C CNN
-F 1 "Arduino_UNO_R3" H 2050 7637 50  0000 C CNN
-F 2 "Footprints:Arduino_UNO_R3" H 2200 5500 50  0001 L CNN
-F 3 "https://www.arduino.cc/en/Main/arduinoBoardUno" H 1850 7600 50  0001 C CNN
-	1    2050 6550
-	-1   0    0    -1
-$EndComp
 $Comp
 L Connector:Conn_01x08_Male J1
@@
 Text GLabel 1250 6500 2    50   Input ~ 0
 GND
-Text GLabel 1250 6600 2    50   Input ~ 0
-VIN
 NoConn ~ 1250 5900
 $Comp
 L Connector:Conn_01x06_Male J2
 U 1 1 5BF499A8
-P 1050 7100
-F 0 "J2" H 1156 7478 50  0000 C CNN
-F 1 "Conn_01x06_Male" H 1156 7387 50  0000 C CNN
-F 2 "Socket_Strips:Socket_Strip_Straight_1x06_Pitch2.54mm" H 1050 7100 50  0001 C CNN
-F 3 "~" H 1050 7100 50  0001 C CNN
-	1    1050 7100
-	1    0    0    -1
-$EndComp
+P 1050 7200
+F 0 "J2" H 1156 7578 50  0000 C CNN
+F 1 "Conn_01x06_Male" H 1156 7487 50  0000 C CNN
+F 2 "Socket_Strips:Socket_Strip_Straight_1x06_Pitch2.54mm" H 1050 7200 50  0001 C CNN
+F 3 "~" H 1050 7200 50  0001 C CNN
+	1    1050 7200
+	1    0    0    1
+$EndComp
+Text GLabel 1250 7400 2    50   Input ~ 0
+A0
+Text GLabel 1250 7300 2    50   Input ~ 0
+A1
+Text GLabel 1250 7200 2    50   Input ~ 0
+A2
+Text GLabel 1250 7100 2    50   Input ~ 0
+A3
+Text GLabel 1250 7000 2    50   Input ~ 0
+A4
 Text GLabel 1250 6900 2    50   Input ~ 0
-A0
-Text GLabel 1250 7000 2    50   Input ~ 0
-A1
-Text GLabel 1250 7100 2    50   Input ~ 0
-A2
-Text GLabel 1250 7200 2    50   Input ~ 0
-A3
-Text GLabel 1250 7300 2    50   Input ~ 0
-A4
-Text GLabel 1250 7400 2    50   Input ~ 0
 A5
 $Comp
 L Connector:Conn_01x08_Male J3
 U 1 1 5BF4A69B
-P 3050 6300
-F 0 "J3" H 3023 6180 50  0000 R CNN
-F 1 "Conn_01x08_Male" H 3023 6271 50  0000 R CNN
-F 2 "Socket_Strips:Socket_Strip_Straight_1x08_Pitch2.54mm" H 3050 6300 50  0001 C CNN
-F 3 "~" H 3050 6300 50  0001 C CNN
-	1    3050 6300
-	-1   0    0    1
-$EndComp
-Text GLabel 2850 5900 0    50   Input ~ 0
+P 2850 7100
+F 0 "J3" H 2823 6980 50  0000 R CNN
+F 1 "Conn_01x08_Male" H 2823 7071 50  0000 R CNN
+F 2 "Socket_Strips:Socket_Strip_Straight_1x08_Pitch2.54mm" H 2850 7100 50  0001 C CNN
+F 3 "~" H 2850 7100 50  0001 C CNN
+	1    2850 7100
+	-1   0    0    -1
+$EndComp
+Text GLabel 2650 7500 0    50   Input ~ 0
 D0
-Text GLabel 2850 6000 0    50   Input ~ 0
+Text GLabel 2650 7400 0    50   Input ~ 0
 D1
-Text GLabel 2850 6100 0    50   Input ~ 0
+Text GLabel 2650 7300 0    50   Input ~ 0
 D2
-Text GLabel 2850 6200 0    50   Input ~ 0
+Text GLabel 2650 7200 0    50   Input ~ 0
 D3
-Text GLabel 2850 6300 0    50   Input ~ 0
+Text GLabel 2650 7100 0    50   Input ~ 0
 D4
-Text GLabel 2850 6400 0    50   Input ~ 0
+Text GLabel 2650 7000 0    50   Input ~ 0
 D5
-Text GLabel 2850 6500 0    50   Input ~ 0
+Text GLabel 2650 6900 0    50   Input ~ 0
 D6
-Text GLabel 2850 6600 0    50   Input ~ 0
+Text GLabel 2650 6800 0    50   Input ~ 0
 D7
 $Comp
 L Connector:Conn_01x10_Male J4
 U 1 1 5BF4AB57
-P 3050 7250
-F 0 "J4" H 3023 7130 50  0000 R CNN
-F 1 "Conn_01x10_Male" H 3023 7221 50  0000 R CNN
-F 2 "Socket_Strips:Socket_Strip_Straight_1x10_Pitch2.54mm" H 3050 7250 50  0001 C CNN
-F 3 "~" H 3050 7250 50  0001 C CNN
-	1    3050 7250
-	-1   0    0    1
-$EndComp
-Text GLabel 2850 6750 0    50   Input ~ 0
+P 2850 6150
+F 0 "J4" H 2823 6030 50  0000 R CNN
+F 1 "Conn_01x10_Male" H 2823 6121 50  0000 R CNN
+F 2 "Socket_Strips:Socket_Strip_Straight_1x10_Pitch2.54mm" H 2850 6150 50  0001 C CNN
+F 3 "~" H 2850 6150 50  0001 C CNN
+	1    2850 6150
+	-1   0    0    -1
+$EndComp
+Text GLabel 2650 6650 0    50   Input ~ 0
 D8
-Text GLabel 2850 6850 0    50   Input ~ 0
+Text GLabel 2650 6550 0    50   Input ~ 0
 D9
-Text GLabel 2850 6950 0    50   Input ~ 0
+Text GLabel 2650 6450 0    50   Input ~ 0
 D10
-Text GLabel 2850 7050 0    50   Input ~ 0
+Text GLabel 2650 6350 0    50   Input ~ 0
 D11
-Text GLabel 2850 7150 0    50   Input ~ 0
+Text GLabel 2650 6250 0    50   Input ~ 0
 D12
-Text GLabel 2850 7250 0    50   Input ~ 0
+Text GLabel 2650 6150 0    50   Input ~ 0
 D13
-Text GLabel 2850 7350 0    50   Input ~ 0
+Text GLabel 2650 6050 0    50   Input ~ 0
 GND
-Text GLabel 2850 7450 0    50   Input ~ 0
+Text GLabel 2650 5950 0    50   Input ~ 0
 AREF
-Text GLabel 2850 7550 0    50   Input ~ 0
+Text GLabel 2650 5850 0    50   Input ~ 0
 SDA
-Text GLabel 2850 7650 0    50   Input ~ 0
+Text GLabel 2650 5750 0    50   Input ~ 0
 SCL
 $Comp
@@
 Wire Wire Line
 	6900 1100 6900 1150
-Text Label 6650 1250 1    50   ~ 0
-VIN
 Text GLabel 5900 1850 0    50   Input ~ 0
 SDA
@@
 	1    0    0    -1
 $EndComp
+NoConn ~ 1250 6600
 $EndSCHEMATC

Commit message: reduce the number of electrolytic capacitors, improve routing
Parts:
- removed C11, C8: 1U ELEC, Capacitors_SMD:CP_Elec_5x5.8, symbol Device:CP
- U1, U2, U3: footprint Footprints:TSSOP-16_4.4x5mm_P0.65mm -> footprints:TSSOP-16_4.4x5mm_P0.65mm
Changed lines of the file:
@@
 EESchema Schematic File Version 4
+LIBS:adc-cache
 EELAYER 26 0
 EELAYER END
@@
 F 0 "U1" H 1750 3378 50  0000 C CNN
 F 1 "ADC128D818" H 1750 3287 50  0000 C CNN
-F 2 "Footprints:TSSOP-16_4.4x5mm_P0.65mm" H 1750 2400 50  0001 C CIN
+F 2 "footprints:TSSOP-16_4.4x5mm_P0.65mm" H 1750 2400 50  0001 C CIN
 F 3 "http://www.ti.com/lit/ds/symlink/adc128d818.pdf" H 1750 2400 50  0001 C CNN
 	1    1750 2400
@@
 F 0 "U3" H 6650 3428 50  0000 C CNN
 F 1 "ADC128D818" H 6650 3337 50  0000 C CNN
-F 2 "Footprints:TSSOP-16_4.4x5mm_P0.65mm" H 6650 2450 50  0001 C CIN
+F 2 "footprints:TSSOP-16_4.4x5mm_P0.65mm" H 6650 2450 50  0001 C CIN
 F 3 "http://www.ti.com/lit/ds/symlink/adc128d818.pdf" H 6650 2450 50  0001 C CNN
 	1    6650 2450
@@
 Wire Wire Line
 	8100 3050 8100 3100
-$Comp
-L Device:CP C11
-U 1 1 5BF7FE39
-P 7600 2900
-F 0 "C11" H 7718 2946 50  0000 L CNN
-F 1 "1U ELEC" H 7718 2855 50  0000 L CNN
-F 2 "Capacitors_SMD:CP_Elec_5x5.8" H 7638 2750 50  0001 C CNN
-F 3 "~" H 7600 2900 50  0001 C CNN
-	1    7600 2900
-	1    0    0    -1
-$EndComp
-Wire Wire Line
-	7150 2750 7600 2750
-Connection ~ 7600 2750
-Wire Wire Line
-	7600 2750 8100 2750
-$Comp
-L power:GND #PWR029
-U 1 1 5BF7FE43
-P 7600 3100
-F 0 "#PWR029" H 7600 2850 50  0001 C CNN
-F 1 "GND" H 7605 2927 50  0000 C CNN
-F 2 "" H 7600 3100 50  0001 C CNN
-F 3 "" H 7600 3100 50  0001 C CNN
-	1    7600 3100
-	1    0    0    -1
-$EndComp
-Wire Wire Line
-	7600 3050 7600 3100
 Text Label 7150 2750 0    50   ~ 0
 VREF
@@
 F 0 "U2" H 5650 6378 50  0000 C CNN
 F 1 "ADC128D818" H 5650 6287 50  0000 C CNN
-F 2 "Footprints:TSSOP-16_4.4x5mm_P0.65mm" H 5650 5400 50  0001 C CIN
+F 2 "footprints:TSSOP-16_4.4x5mm_P0.65mm" H 5650 5400 50  0001 C CIN
 F 3 "http://www.ti.com/lit/ds/symlink/adc128d818.pdf" H 5650 5400 50  0001 C CNN
 	1    5650 5400
@@
 Wire Wire Line
 	7100 6000 7100 6050
-$Comp
-L Device:CP C8
-U 1 1 5BFE9A56
-P 6600 5850
-F 0 "C8" H 6718 5896 50  0000 L CNN
-F 1 "1U ELEC" H 6718 5805 50  0000 L CNN
-F 2 "Capacitors_SMD:CP_Elec_5x5.8" H 6638 5700 50  0001 C CNN
-F 3 "~" H 6600 5850 50  0001 C CNN
-	1    6600 5850
-	1    0    0    -1
-$EndComp
-Wire Wire Line
-	6150 5700 6600 5700
-Connection ~ 6600 5700
-Wire Wire Line
-	6600 5700 7100 5700
-$Comp
-L power:GND #PWR020
-U 1 1 5BFE9A60
-P 6600 6050
-F 0 "#PWR020" H 6600 5800 50  0001 C CNN
-F 1 "GND" H 6605 5877 50  0000 C CNN
-F 2 "" H 6600 6050 50  0001 C CNN
-F 3 "" H 6600 6050 50  0001 C CNN
-	1    6600 6050
-	1    0    0    -1
-$EndComp
-Wire Wire Line
-	6600 6000 6600 6050
 Text Label 6150 5700 0    50   ~ 0
 VREF
@@
 $EndComp
 NoConn ~ 1250 6600
+Wire Wire Line
+	7150 2750 8100 2750
+Wire Wire Line
+	6150 5700 7100 5700
 $EndSCHEMATC
